Commit message: add odom frame

File: racecar.xacro (robot description, xacro)
@@ -17,4 +17,10 @@
     <color rgba="0.3 0.57 1. 1."/>
   </material>
+  <link name="base_footprint"/>
+  <joint name="base_joint" type="fixed">
+    <parent link="base_footprint"/>
+    <child link="base_link" />
+    <origin xyz="0 0.0 0.07" rpy="0 0 0.0"/>
+  </joint>
   <link name="base_link">
     <visual>
@@ -26,10 +32,10 @@
     </visual>
   </link>
-  <joint name="base_to_laser_model" type="fixed">
+  <joint name="base_to_scan" type="fixed">
     <parent link="base_link"/>
-    <child link="laser_model"/>
+    <child link="base_scan"/>
     <origin xyz="${laser_distance_from_base_link} 0 ${ground_offset+height+(laser_height/2)}"/>
   </joint>
-  <link name="laser_model">
+  <link name="base_scan">
     <visual>
       <geometry>

Commit message: EDIT:Odom Frame

File: racecar.xacro (robot description, xacro)
@@ -21,5 +21,5 @@
     <parent link="base_footprint"/>
     <child link="base_link" />
-    <origin xyz="0 0.0 0.07" rpy="0 0 0.0"/>
+    <origin xyz="0 0.0 0.0" rpy="0 0 0.0"/>
   </joint>
   <link name="base_link">

Commit message: Final:Setting

File: racecar.xacro (robot description, xacro)
@@ -17,11 +17,11 @@
     <color rgba="0.3 0.57 1. 1."/>
   </material>
-  <link name="base_footprint"/>
+  <!-- <link name="base_footprint"/>
   <joint name="base_joint" type="fixed">
     <parent link="base_footprint"/>
     <child link="base_link" />
-    <origin xyz="0 0.0 0.0" rpy="0 0 0.0"/>
-  </joint>
-  <link name="base_link">
+    <origin xyz="0.0 0.0 0.0" rpy="0 0 0.0"/>
+  </joint> -->
+  <link name="base_footprint">
     <visual>
       <origin xyz="${wheelbase/2} 0 ${ground_offset+height/2}"/>
@@ -33,5 +33,5 @@
   </link>
   <joint name="base_to_scan" type="fixed">
-    <parent link="base_link"/>
+    <parent link="base_footprint"/>
     <child link="base_scan"/>
     <origin xyz="${laser_distance_from_base_link} 0 ${ground_offset+height+(laser_height/2)}"/>
@@ -46,5 +46,5 @@
   </link>
   <joint name="base_to_back_left_wheel" type="fixed">
-    <parent link="base_link"/>
+    <parent link="base_footprint"/>
     <child link="back_left_wheel"/>
     <origin xyz="0 ${(wheel_length+width)/2} ${wheel_radius}"/>
@@ -60,5 +60,5 @@
   </link>
   <joint name="base_to_back_right_wheel" type="fixed">
-    <parent link="base_link"/>
+    <parent link="base_footprint"/>
     <child link="back_right_wheel"/>
     <origin xyz="0 ${-(wheel_length+width)/2} ${wheel_radius}"/>
@@ -74,5 +74,5 @@
   </link>
   <joint name="base_to_front_left_hinge" type="fixed">
-    <parent link="base_link"/>
+    <parent link="base_footprint"/>
     <child link="front_left_hinge"/>
     <origin xyz="${wheelbase} ${(wheel_length+width)/2} ${wheel_radius}"/>
@@ -93,5 +93,5 @@
   </link>
   <joint name="base_to_front_right_hinge" type="fixed">
-    <parent link="base_link"/>
+    <parent link="base_footprint"/>
     <child link="front_right_hinge"/>
     <origin xyz="${wheelbase} ${-(wheel_length+width)/2} ${wheel_radius}"/>

Commit message: Final:Set

File: racecar.xacro (robot description, xacro)
@@ -17,11 +17,11 @@
     <color rgba="0.3 0.57 1. 1."/>
   </material>
-  <!-- <link name="base_footprint"/>
+  <link name="base_footprint"/>
   <joint name="base_joint" type="fixed">
     <parent link="base_footprint"/>
     <child link="base_link" />
     <origin xyz="0.0 0.0 0.0" rpy="0 0 0.0"/>
-  </joint> -->
-  <link name="base_footprint">
+  </joint>
+  <link name="base_link">
     <visual>
       <origin xyz="${wheelbase/2} 0 ${ground_offset+height/2}"/>
@@ -33,5 +33,5 @@
   </link>
   <joint name="base_to_scan" type="fixed">
-    <parent link="base_footprint"/>
+    <parent link="base_link"/>
     <child link="base_scan"/>
     <origin xyz="${laser_distance_from_base_link} 0 ${ground_offset+height+(laser_height/2)}"/>
@@ -46,5 +46,5 @@
   </link>
   <joint name="base_to_back_left_wheel" type="fixed">
-    <parent link="base_footprint"/>
+    <parent link="base_link"/>
     <child link="back_left_wheel"/>
     <origin xyz="0 ${(wheel_length+width)/2} ${wheel_radius}"/>
@@ -60,5 +60,5 @@
   </link>
   <joint name="base_to_back_right_wheel" type="fixed">
-    <parent link="base_footprint"/>
+    <parent link="base_link"/>
     <child link="back_right_wheel"/>
     <origin xyz="0 ${-(wheel_length+width)/2} ${wheel_radius}"/>
@@ -74,5 +74,5 @@
   </link>
   <joint name="base_to_front_left_hinge" type="fixed">
-    <parent link="base_footprint"/>
+    <parent link="base_link"/>
     <child link="front_left_hinge"/>
     <origin xyz="${wheelbase} ${(wheel_length+width)/2} ${wheel_radius}"/>
@@ -93,5 +93,5 @@
   </link>
   <joint name="base_to_front_right_hinge" type="fixed">
-    <parent link="base_footprint"/>
+    <parent link="base_link"/>
     <child link="front_right_hinge"/>
     <origin xyz="${wheelbase} ${-(wheel_length+width)/2} ${wheel_radius}"/>
